File: Dodobot/Dodobot.sch (EAGLE design)
At the start: 49 parts, among them Q1 2N3904, Q2 2N3904, Q3 2N7000, Q4 2N7000

Commit message: Restoring Rev 2 changes
Adding stepper encoder
Increased tracewidth size
Added VIN trace to teensy
changed from 40-pin bus to 3 pin header
Parts:
- removed D4: (no value), SparkFun-LED:LED1206
- removed JP1, JP2: JUMPER-SMT_2_NO_NO-SILK, SparkFun-Jumpers:JUMPER-SMT_2_NO_NO-SILK
- removed JP3, JP4: JUMPER-SMT_2_NC_TRACE_NO-SILK, SparkFun-Jumpers:JUMPER-SMT_2_NC_TRACE_NO-SILK
- removed MAIN_HEADER: (no value), adafruit:PINHD-2X20
- removed R12: WSLP1206R0500FEA, Resistor_Capacitor:WSLP1206R0500FEA
- removed R7, R8: CRCW08050000Z0EA, Resistor_Capacitor:CRCW08050000Z0EA
- added BUMP: 0705530003, Molex Right Angle 4 position 0705530003:0705530003
- added JETSON_PWR: 1935161, 1935161:1935161
- added STEP_ENC: 0705530004, Molex Right Angle 4 position 0705530003:0705530004
- JETSON: value 1935161 -> (none); device 1935161:1935161 -> pinhead:PINHD-1X3
Connections:
- removed net N$12: JP4.1, U$1.14/A0
- removed net N$13: JP3.2, U$1.24
- removed net N$15: JP2.1, MAIN_HEADER.12
- removed net N$4: D4.A, R12.1
- removed net N$5: JP1.2, MAIN_HEADER.11
- removed net N$6: Q2.E, R7.2
- removed net N$7: Q1.E, R8.2
- removed net RX_RPI: MAIN_HEADER.10, U$1.33/A14
- removed net SERVO3: SERVOS.12, U$1.3/CANTX
- removed net SERVO4: SERVOS.9, U$1.5
- removed net STATUS_LED: MAIN_HEADER.14, R12.2
- removed net TX_RPI: MAIN_HEADER.8, U$1.34/A15
- new net BUMP1: BUMP.1, U$1.3/CANTX
- new net BUMP2: BUMP.3, U$1.5
- new net RX_JETSON: JETSON.1, U$1.33/A14
- new net STEP_ENCA: STEP_ENC.3, U$1.31/A12
- new net STEP_ENCB: STEP_ENC.1, U$1.32/A13
- new net TX_JETSON: JETSON.2, U$1.34/A15
- net +5V: now also JETSON_PWR.1, U$1.VIN; no longer JETSON.1
- net BUTTON_LED: now also U$1.14/A0; no longer JP2.2, JP4.2
- net GND: now also BUMP.2, BUMP.4, JETSON.3, JETSON_PWR.2, Q1.E, Q2.E, SERVOS.12, SERVOS.9, STEP_ENC.5; no longer D4.C, JETSON.2, MAIN_HEADER.6, R7.1, R8.1, SERVOS.10, SERVOS.7
- net LATCH_STAT: no longer MAIN_HEADER.13
- net M_STBY: now also U$1.A21/DAC0
- net SERVO1: now also SERVOS.10; no longer SERVOS.1
- net SERVO2: now also SERVOS.7; no longer SERVOS.4
- net TIC_RX: now also U$1.1/TX; no longer U$1.32/A13
- net TIC_TX: now also U$1.0/RX; no longer U$1.31/A12
- net UNLATCH: now also U$1.24; no longer JP1.1, JP3.1
- net VCC: now also STEP_ENC.2
Other:
- note added: "+12V: 12V regulator output"
- note added: "+5V: 5V regulator output"
- note added: "12V regulator"
- note added: "5V regulator"
- note added: "6V regulator"
- note added: "V+: 6V regulator output"
- note removed: "5+: Regular 2 5V output. Goes to RPi"
- note removed: "V+: Regulator 1 5V output, power circuit 1, (main motors, lidar)"

Commit message: minor fixes. Correcting errors in library files
Parts:
- 12V_REG: value S18V20FX -> ELEC-169
- 5V_REG: value D24V50F5 -> ELEC-154
- 6V_REG: value D36V50FX -> ELEC-153
- BATTERY_MONITOR: value INA219 -> ELEC-133
- C1, C2: value FK24X5R0J226M -> 22uF
- MOTOR_DRIVER: value ADAFRUIT_TB6612 -> ELEC-134
- R1, R14, R2, R3, R4, R5: value CRCW08050000Z0EA -> 10K
- R10, R11: value WSLP1206R0500FEA -> 20
- R13: value CRCW08050000Z0EA -> 6K
- R6: value CRCW08050000Z0EA -> 100K
- R9: value (none) -> 10
- renumbered U$3 to MOTOR_DRIVER, U$4 to BATTERY_MONITOR, U$5 to 5V_REG, U$6 to 12V_REG, U$7 to 6V_REG
Connections:
- net GND: now also 12V_REG.GND_IN2
Other:
- note added: "Connector to IR receiver ELEC-150"
- note added: "Connector to ST7735 Display ELEC-102"
- note added: "Connector to Tic T500 Board ELEC-186"
- note added: "Connector to stepper encoder ENC4109 MECH-177"
- note added: "ELEC-135"
- note added: "ELEC-149"
- note added: "Plug to Jetson GPIO Header MECH-101"
- note removed: "12V regulator"
- note removed: "5V regulator"
- note removed: "6V regulator"
